File: Minimal_Prototype_Function_Generator_V0.1/ADM7160ACPZN3.3.kicad_sch (KiCad schematic)
At the start: 4 parts, among them IC3 ADM7160ACPZN3.3-R7

Commit message: new pcb version
Parts:
- +3V3_1: footprint TestPoint:TestPoint_Loop_D3.80mm_Drill2.5mm -> Insyte_Footprints:Testpoint_hole
- C4, C5: footprint Capacitor_SMD:C_0603_1608Metric -> Insyte_Footprints:C_0603
