File: Minimal_Prototype_Function_Generator_V0.1/Power.kicad_sch (KiCad schematic)
At the start: 2 parts

Commit message: new pcb version
Parts:
- removed FB3, FB4: 1.8K OHM AT 100MEGHZ, Inductor_SMD:L_0603_1608Metric, symbol Device:FerriteBead_Small
- added R56, R57: 0R, Insyte_Footprints:R_0603, symbol Device:R
Connections:
- net ADM7160ACPZN3.3_1/+3V3: now also R56.1, R57.1
- net CLKVDD: now also R57.2
- net DVDD: now also R56.2
