File: Minimal_Prototype_Function_Generator_V0.1/STM32.kicad_sch (KiCad schematic)
At the start: 25 parts, among them IC9 STM32L476VGT6, J10 SPI_TP_1, J7 DEBUG_UART_TP_1, J8 I2C_TP1, Y2 ECS-.327-7-16-C-TR

Commit message: new pcb version
Parts:
- C31, C32, C57, C58, C59, C60, C61, C62, C63, C64, C65, C66: footprint Capacitor_SMD:C_0603_1608Metric -> Insyte_Footprints:C_0603
- J10, J7, J8: now not fitted
- R46, R47, R48, R49, R50: footprint Resistor_SMD:R_0603_1608Metric -> Insyte_Footprints:R_0603
- U4: value ~ -> (none)
Connections:
- net CLOCK_EN: now reaches IC9.35 (PB0)
- net CLOCK_SEL: now reaches IC9.36 (PB1)
- no-connect marks 68 -> 66

Commit message: removed lock files
Parts:
- removed U4: (no value), Insyte_Logo_Footprints:15x6_Insyte_Logo, symbol Insyte:Logo
Changed lines of the file:
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@@
-	)
-	(symbol
-		(lib_id "Insyte:Logo")
-		(at 194.31 146.05 0)
-		(unit 1)
-		(body_style 1)
-		(exclude_from_sim no)
-		(in_bom yes)
-		(on_board yes)
-		(in_pos_files yes)
-		(dnp no)
-		(fields_autoplaced yes)
-		(property "Reference" "U4"
-			(at 198.12 144.7799 0)
-			(show_name no)
-			(do_not_autoplace no)
-			(effects
-				(font
-					(size 1.27 1.27)
-				)
-				(justify left)
-			)
-		)
-		(property "Value" ""
-			(at 198.12 147.3199 0)
-			(show_name no)
-			(do_not_autoplace no)
-			(effects
-				(font
-					(size 1.27 1.27)
-				)
-				(justify left)
-			)
-		)
-		(property "Footprint" "Insyte_Logo_Footprints:15x6_Insyte_Logo"
-			(at 194.31 146.05 0)
-			(hide yes)
-			(show_name no)
-			(do_not_autoplace no)
-			(effects
-				(font
-					(size 1.27 1.27)
-				)
-			)
-		)
-		(property "Datasheet" ""
-			(at 194.31 146.05 0)
-			(hide yes)
-			(show_name no)
-			(do_not_autoplace no)
-			(effects
-				(font
-					(size 1.27 1.27)
-				)
-			)
-		)
-		(property "Description" ""
-			(at 194.31 146.05 0)
-			(hide yes)
-			(show_name no)
-			(do_not_autoplace no)
-			(effects
-				(font
-					(size 1.27 1.27)
-				)
-			)
-		)
-		(instances
-			(project "Minimal_Prototype_Function_Generator_V0.1"
-				(path "/4f62c91b-90a7-42e6-9468-9a44c0d5e9c2/41d5001e-a8ed-4e44-9ec1-df5bd6f03dd6"
-					(reference "U4")
-					(unit 1)
-				)
-			)
-		)
 	)
 	(symbol
