File: Minimal_Prototype_Function_Generator_V0.1/AD9106.kicad_sch (KiCad schematic)
At the start: 30 parts, among them IC1 AD9106BCPZ, J1 142-0701-201, T1 ADT2-1T+, Y1 AX3DCF1-156.2500T

Commit message: new pcb version
Parts:
- removed J1: 142-0701-201, Insyte_Footprints:1420701201, symbol 142-0701-201:142-0701-201
- removed JP1, JP2: Jumper_3_Open, Connector_PinHeader_2.54mm:PinHeader_1x03_P2.54mm_Vertical, symbol Jumper:Jumper_3_Open
- removed R4: 100R, Resistor_SMD:R_0603_1608Metric, symbol Device:R
- removed T1: ADT2-1T+, Insyte_Footprints:ADT21T, symbol ADT2-1T+:ADT2-1T+
- added C70, C71: 100nF, Insyte_Footprints:C_0603, symbol Device:C
- added IC5: TMUXHS221FRSWR, Insyte_Footprints:TMUXHS221FRSWR, symbol TMUXHS221FRSWR:TMUXHS221FRSWR
- added J12: 142-0701-801, Insyte_Footprints:142-0701-851, symbol 142-0701-801:142-0701-801
- added R59: 39K, Insyte_Footprints:R_0603, symbol Device:R
- added R60, R62: 100R, Insyte_Footprints:R_0603, symbol Device:R
- added R61: 50R, Insyte_Footprints:R_0603, symbol Device:R
- C1, C10, C17, C18, C9: footprint Capacitor_SMD:C_0603_1608Metric -> Insyte_Footprints:C_0402
- C11, C12, C13, C14, C15, C16, C19, C20, C21, C22: footprint Capacitor_SMD:C_0603_1608Metric -> Insyte_Footprints:C_0603
- C6, C7, C8: value 0.1uF -> 100nF; footprint Capacitor_SMD:C_0603_1608Metric -> Insyte_Footprints:C_0603
- R5, R6, R7, R8, R9: footprint Resistor_SMD:R_0603_1608Metric -> Insyte_Footprints:R_0603
Connections:
- net CLKN: now also IC5.2 (D-)
- net CLKP: now also IC5.1 (D+)
- net CLKVDD: now also C71.2, IC5.9 (VCC)
- net GND: now also C70.1, C71.1, IC5.3 (GND), J12.2, J12.3 (Ext), J12.4 (Ext), J12.5 (Ext), R59.2, R61.1
- net at C7.2: now also IC5.5 (D1+)
- net at C8.2: now also IC5.4 (D1-)
- net at C7.1, Y1.4 (OUTPUT): now also R62.1
- net at C8.1, Y1.5 (COMP_OUT): now also R62.2
- new net: C70.2, IC5.6 (D2-), R59.1
- new net: IC5.7 (D2+), R60.2
- new net: J12.1, R60.1, R61.2
- new net CLOCK_EN: IC5.8 (OEN)
- new net CLOCK_SEL: IC5.10 (SEL)
- no-connect marks 1 -> 0
Other:
- note removed: "Connect this terminal and above terminal in same position! Pos 2-3 on board crystal Pos 2-3 external trigger"
- moved on the sheet: C6, C7, C8, Y1

Commit message: V2.0
Parts:
- J12: value 142-0701-801 -> SMA-J-P-H-ST-EM1
Connections:
- net GND: no longer J12.4 (Ext), J12.5 (Ext)
Changed lines of the file:
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@@
 			)
 		)
-		(property "Value" "142-0701-801"
+		(property "Value" "SMA-J-P-H-ST-EM1"
 			(at 29.718 83.058 0)
 			(show_name no)
@@
 		(pin "3"
 		)
-		(pin "5"
-		)
-		(pin "4"
-		)
 		(instances
