File: Minimal_Prototype_Function_Generator_V0.1/LT3472EDD.kicad_sch (KiCad schematic)
At the start: 18 parts, among them IC4 LT3472EDD#PBF, P5V2_TP1 TestPoint

Commit message: new pcb version
Parts:
- removed FB1, FB2: 1.8K OHM AT 100MEGHZ, Inductor_SMD:L_0603_1608Metric, symbol Device:FerriteBead_Small
- added R54, R55: 0R, Insyte_Footprints:R_0603, symbol Device:R
- C23, C25, C26, C27, C28, C29, C30: footprint Capacitor_SMD:C_0603_1608Metric -> Insyte_Footprints:C_0603
- C24: footprint Capacitor_SMD:C_0603_1608Metric -> Insyte_Footprints:C_0402
- N5V2_TP1, P5V2_TP1: footprint TestPoint:TestPoint_Loop_D3.80mm_Drill2.5mm -> Insyte_Footprints:Testpoint_hole
- R11, R12: footprint Resistor_SMD:R_0603_1608Metric -> Insyte_Footprints:R_0603
Connections:
- net N5V2: now also R55.2
- net N5V2_VN: now also L4.1, L4.3, R55.1
- net P5V2: now also R54.2
- net P5V2_VP: now also R54.1; no longer L4.1, L4.3
Other:
- moved on the sheet: C23
