File: Minimal_Prototype_Function_Generator_V0.1/Minimal_Prototype_Function_Generator_V0.1.kicad_sch (KiCad schematic)
At the start: 3 parts, among them J6 142-0701-201

Commit message: new pcb version
Parts:
- removed J6: 142-0701-201, Insyte_Footprints:1420701201, symbol 142-0701-201:142-0701-201
- added J13: 142-0701-801, Insyte_Footprints:142-0701-851, symbol 142-0701-801:142-0701-801
- R10, R45: footprint Resistor_SMD:R_0603_1608Metric -> Insyte_Footprints:R_0603
Connections:
- net GND: now also J13.2, J13.3 (Ext), J13.4 (Ext), J13.5 (Ext)
- net at R45.2: now also J13.1
Other:
- sheet Function Generator ports: added CLOCK_EN, CLOCK_SEL; removed none
- sheet STM32 ports: added CLOCK_EN, CLOCK_SEL; removed none
- note added: "- FB1 & FB2 replaced with 0R resistors - Connect pin 2 of L4 to N5V2_VN instead of P5V2_VP - Removed unneeded TVS diode on CC1 and CC2 lines."

Commit message: V2.0
Parts:
- J13: value 142-0701-801 -> SMA-J-P-H-ST-EM1
Connections:
- net GND: no longer J13.4 (Ext), J13.5 (Ext)
Changed lines of the file:
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@@
 			)
 		)
-		(property "Value" "142-0701-801"
+		(property "Value" "SMA-J-P-H-ST-EM1"
 			(at 168.148 110.998 0)
 			(show_name no)
@@
 		(pin "3"
 		)
-		(pin "5"
-		)
-		(pin "4"
-		)
 		(instances
