File: Minimal_Prototype_Function_Generator_V0.1/Output_Stage.kicad_sch (KiCad schematic)
At the start: 4 parts, among them J2 142-0701-201, J3 142-0701-201, J4 142-0701-201, J5 142-0701-201

Commit message: new pcb version
Parts:
- removed J2, J3, J4, J5: 142-0701-201, Insyte_Footprints:1420701201, symbol 142-0701-201:142-0701-201
- added J14, J15, J16, J17: 142-0701-801, Insyte_Footprints:142-0701-851, symbol 142-0701-801:142-0701-801
Connections:
- net GND: now also J14.2, J14.3 (Ext), J14.4 (Ext), J14.5 (Ext), J15.2, J15.3 (Ext), J15.4 (Ext), J15.5 (Ext), J16.2, J16.3 (Ext), J16.4 (Ext), J16.5 (Ext), J17.2, J17.3 (Ext), J17.4 (Ext), J17.5 (Ext)
- net Op_Amp_1/AMP1_OUT: now also J15.1
- net Op_Amp_1/AMP_OUT: now also J14.1
- net Op_Amp_2/AMP1_OUT: now also J17.1
- net Op_Amp_2/AMP_OUT: now also J16.1

Commit message: V2.0
Parts:
- J14, J15, J16, J17: value 142-0701-801 -> SMA-J-P-H-ST-EM1
Connections:
- net GND: no longer J14.4 (Ext), J14.5 (Ext), J15.4 (Ext), J15.5 (Ext), J16.4 (Ext), J16.5 (Ext), J17.4 (Ext), J17.5 (Ext)
Changed lines of the file:
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@@
 			)
 		)
-		(property "Value" "142-0701-801"
+		(property "Value" "SMA-J-P-H-ST-EM1"
 			(at 108.712 65.278 0)
 			(show_name no)
@@
 		)
 		(pin "3"
-		)
-		(pin "4"
-		)
-		(pin "5"
 		)
 		(instances
@@
 			)
 		)
-		(property "Value" "142-0701-801"
+		(property "Value" "SMA-J-P-H-ST-EM1"
 			(at 115.062 28.448 0)
 			(show_name no)
@@
 		)
 		(pin "3"
-		)
-		(pin "4"
-		)
-		(pin "5"
 		)
 		(instances
@@
 			)
 		)
-		(property "Value" "142-0701-801"
+		(property "Value" "SMA-J-P-H-ST-EM1"
 			(at 115.062 62.738 0)
 			(show_name no)
@@
 		)
 		(pin "3"
-		)
-		(pin "5"
-		)
-		(pin "4"
 		)
 		(instances
@@
 			)
 		)
-		(property "Value" "142-0701-801"
+		(property "Value" "SMA-J-P-H-ST-EM1"
 			(at 108.712 30.988 0)
 			(show_name no)
@@
 		(pin "3"
 		)
-		(pin "4"
-		)
-		(pin "5"
-		)
 		(instances
