File: Minimal_Prototype_Function_Generator_V0.1/USB_C.kicad_sch (KiCad schematic)
At the start: 8 parts, among them J9 USB4500-03-0-A

Commit message: new pcb version
Parts:
- removed D4: SM05.TCT, Insyte_Footprints:SOT95P237X125-3N, symbol Power_Protection:SP0502BAHT
- D6: footprint Insyte_Footprints:LEDC1608X85N -> Insyte_Footprints:CSL1901MW1
- R51, R52, R53: footprint Resistor_SMD:R_0603_1608Metric -> Insyte_Footprints:R_0603

Commit message: V2.0
Parts:
- R53: value 325R -> 500R
Changed lines of the file:
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@@
 	(text "ESD"
 		(exclude_from_sim no)
-		(at 109.982 16.764 0)
+		(at 106.934 17.272 0)
 		(effects
 			(font
@@
 			)
 		)
-		(property "Value" "325R"
+		(property "Value" "500R"
 			(at 207.01 31.7499 0)
 			(show_name no)
@@
 			(show_name no)
 			(do_not_autoplace no)
+			(effects
+				(font
+					(size 1.27 1.27)
+				)
+			)
+		)
+		(property "manf#" ""
+			(at 204.47 30.48 0)
+			(hide yes)
+			(show_name no)
+			(do_not_autoplace no)
+			(effects
+				(font
+					(size 1.27 1.27)
+				)
+			)
+		)
+		(property "LCSC" ""
+			(at 204.47 30.48 0)
+			(hide yes)
+			(show_name no)
+			(do_not_autoplace no)
+			(effects
+				(font
+					(size 1.27 1.27)
+				)
+			)
+		)
+		(property "kicost:pricing" ""
+			(at 204.47 30.48 0)
+			(hide yes)
+			(show_name no)
+			(do_not_autoplace no)
